File: sensors/lightning_detector/schematic/lightning_detector.kicad_pcb (KiCad board)
At the start: 2 copper layers, 70.9 x 44.9 mm, 30 parts, among them J1 CJMCU-3935, J2 boot, J3 VEML7700, J4 jst, J5 AS7731, J6 CJMCU-3935, Q2 Q_PNP_BEC, Q3 Q_PMOS_GSD, Q4 Q_PNP_BEC, U1 ESP32-WROOM-32, U2 TPS7A0533PDBZR, U3 TL431DBZ

Commit message: update sensor schematics
Other:
- net class Default removed
