File: sensors/temperature_pressure_humidity_gas/schematic/temperature_pressure_humidity_gas.kicad_pcb (KiCad board)
At the start: 2 copper layers, 38.5 x 51.9 mm, 37 parts, among them J1 Power Input (12/24), J2 boot, J4 jst, Q1 Q_PMOS_GSD, U1 ESP32-WROOM-32, U2 ADP2303ARDZ, U3 TPS7133, U4 BME680, U5 2.5v, U6 1.24v

Commit message: update sensor schematics
Other:
- net class Default removed
