File: sensors/wind_transmitter/schematic/anemometer_board.kicad_pcb (KiCad board)
At the start: 4 copper layers, 277.9 x 24 mm, 41 parts, among them J1 Conn_02x03_Odd_Even, J2 Conn_01x04, J3 Conn_02x03_Odd_Even, U1 SC2402, U2 MT6816

Commit message: update sensor schematics
Other:
- net class Default removed
